File: resources/circuit/aeroPi.kicad_pcb (KiCad board)
At the start: 2 copper layers, 65 x 56.5 mm, 75 parts, among them J1 CONN_COAXIAL, J2 CONN_01X03, J3 CONN_01X04, J4 CONN_01X03, J5 CONN_01X03, M0 MountingHole_3mm, M1 MountingHole_3mm, M2 MountingHole_3mm, M3 MountingHole_3mm, P1 CONN_01X02, P2 CONN_01X02, P3 Raspberry_Pi_+_Conn, P4 CONN_01X02, Q1 BSS138, Q2 BSS138, Q3 BSS138, Q4 BSS138, Q5 BSS138, U1 MIC5219-3.3BM5, U11 MAP Pressure, U12 LM358, U2 CAT24C32HU4I-GT3, U3 BME280, U5 DMMT5401, U6 FGPMMOPA6H, U7 MPU-9250, U8 Airspeed, U9 ADS7828

Commit message: Work on circuit and add documentation + 3D model
Parts:
- removed C4: 0.1uf, Capacitors_SMD:C_0603
- removed J3: CONN_01X04, Pin_Headers:Pin_Header_Straight_1x04_Pitch2.54mm
- removed J5: CONN_01X03, Pin_Headers:Pin_Header_Straight_1x03_Pitch2.54mm
- removed JP1: JUMPER, Resistors_SMD:R_0603
- removed P1: CONN_01X02, Pin_Headers:Pin_Header_Straight_1x02_Pitch2.54mm
- removed Q1: BSS138, TO_SOT_Packages_SMD:SOT-23
- removed R11: 10k, Resistors_SMD:R_0603
- removed R12: 47k, Resistors_SMD:R_0603
- removed R3, R5: 3.9k, Resistors_SMD:R_0603
- removed U2: CAT24C32HU4I-GT3, w_smd_dil:tssop-8
- removed U5: DMMT5401, w_smd_trans:sot23-6
- added D1: 1N4148, Diodes_SMD:D_SOD-323, F.Cu at (123.9, 96.6)
- BT1: footprint Connectors:CR1220 -> Battery_Holders:Keystone_3000_1x12mm-CoinCell
- D4: value Diode -> 1N4007; footprint Diodes_SMD:D_0603 -> Diodes_SMD:D_SOD-323
- J2: value CONN_01X03 -> DB15_FEMALE; footprint Pin_Headers:Pin_Header_Straight_1x03_Pitch2.54mm -> Connectors:DB15FC
- J4: value CONN_01X03 -> CONN_01X04; footprint Pin_Headers:Pin_Header_Straight_1x03_Pitch2.54mm -> Pin_Headers:Pin_Header_Straight_1x04_Pitch2.54mm
- R1: value 1k -> 10K
- U11: footprint SMD_Packages:SOIC-8-N -> aeroPi:MPXA6115A
- U8: footprint SMD_Packages:SOIC-8-N -> aeroPi:MPXV5004DP
- moved J1 47.1 mm to (113.6, 82.9), turned to 180 degrees
- moved P2 42.8 mm to (154.9, 98.7), turned to 0 degrees
- moved C10 38.7 mm to (155.9, 89.2), turned to 0 degrees
- moved C3 38.2 mm to (152.2, 100.5), turned to 90 degrees
- moved J2 35.8 mm to (139.1, 122.3), turned to 180 degrees
- moved R1 35.4 mm to (127.5, 96.6), turned to 0 degrees
- moved U1 35.3 mm to (149.4, 100.3), turned to 180 degrees
- moved U7 34.2 mm to (154.2, 92.1), turned to 180 degrees
- moved C5 33.6 mm to (149.5, 89.0), turned to 90 degrees
- moved C1 32.8 mm to (148.0, 89.0), turned to 90 degrees
- moved C13 32.5 mm to (152.6, 89.2), turned to 0 degrees
- moved C7 32.2 mm to (146.6, 100.5), turned to 90 degrees
- moved U3 29.1 mm to (148.5, 92.1), turned to 270 degrees
- moved C12 28.7 mm to (151.3, 91.8), turned to 270 degrees
- moved R20 27.7 mm to (126.7, 115.6)
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Connections:
- J2 pad 1: Net-(J2-Pad1) -> /Tachometer
- J2 pad 2: GND -> /Fuel_Flow_In
- J2 pad 3: /+5V -> /VoltageMeter
- J4 pad 1: GND -> /I2C_SCLK
- J4 pad 2: /CurrentMeter -> /I2C_SDA
- J4 pad 3: /+5V -> /+3.3V
- P3 pad 11: (no net) -> /Fuel_Flow
- P3 pad 12: (no net) -> /Tach
- P3 pad 2: /Back Power Protection/5V_MCU -> /+5VRpi
- P3 pad 22: /Fuel_Flow -> (no net)
- P3 pad 27: Net-(P3-Pad27) -> (no net)
- P3 pad 28: Net-(P3-Pad28) -> (no net)
- P3 pad 29: /1PPS -> (no net)
- P3 pad 4: /Back Power Protection/5V_MCU -> /+5VRpi
- P3 pad 7: /Tach -> /1PPS
- Q5 pad 3: Net-(J2-Pad1) -> /Fuel_Flow_In
- R1 pad 1: /+3.3V -> Net-(D1-Pad2)
- R1 pad 2: Net-(JP1-Pad1) -> /+3.3V
- R30 pad 2: Net-(J2-Pad1) -> /Fuel_Flow_In
- U6 pad 10: /TXD -> Net-(D1-Pad2)
- U6 pad 9: /RXD -> /TXD
- U9 pad 8: (no net) -> /AirTemp
Routing:
- net /+3.3V: track 133.4 -> 80.7 mm
- net /+5V: track 168.1 -> 118.9 mm, vias 2 -> 1
- net /MAP: track 12.1 -> 46.4 mm
- net Net-(P3-Pad28): track 26.6 -> 0.00 mm, vias 2 -> 0
- net /Fuel_Flow_In: track 0.00 -> 26.3 mm, vias 0 -> 2
- net Net-(D1-Pad2): track 0.00 -> 26.3 mm, vias 0 -> 2
- net Net-(P3-Pad27): track 25.1 -> 0.00 mm, vias 2 -> 0
- net /1PPS: track 36.1 -> 12.8 mm, vias 1 -> 2
- net /VBACKUP: track 21.6 -> 40.2 mm, vias 0 -> 2
- net /Fuel_Flow: track 13.8 -> 31.9 mm, vias 1 -> 2
- net /I2C_SCLK: track 75.5 -> 58.8 mm, vias 3 -> 4
- net /AirTemp: track 0.00 -> 15.0 mm
- net /I2C_SDA: track 82.0 -> 67.1 mm, vias 3 -> 0
- net /Back Power Protection/5V_MCU: track 14.1 -> 0.00 mm
- net /RXD: track 44.1 -> 57.2 mm, vias 2 -> 1
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- removed copper zone on F.Cu, net Net-(R11-Pad1)
Other:
- board text added: "3v3"
- board text added: "SCL"
- board text added: "SDA"
- board text added: "aeroPi © CD System 2017 V1.0"
- board text removed: "+5V Gnd Sig Flow meter"
- board text removed: "+5V Sig Gnd"
- board text removed: "+Vcc 8V - 40V"
- board text removed: "A. meter"
- board text removed: "CD System"
- board text removed: "Display Power +5V Gnd"
- board text removed: "Gnd"
- board text removed: "Oil Press Oil Temp CHT Tach"
- board text removed: "V. meter"
