File: resources/circuit/aeroPi.sch (KiCad schematic (older format))
At the start: 72 parts, among them J1 CONN_COAXIAL, J2 Screw_Terminal_1x12, P1 CONN_01X02, P2 CONN_01X02, P3 Raspberry_Pi_+_Conn, U1 LM3489, U10 Airspeed, U11 Static Pressure, U12 MAP Pressure, U2 CAT24C32HU4I-GT3, U3 FDC5614P, U4 LM1117IMPX-ADJ, U6 FGPMMOPA6H, U7 MPU-9250, U8 MCP3008BIS, U9 MCP3008BIS

Commit message: Work on schematic & PCB
Parts:
- U10: symbol MPXA6115A -> MPXV5004DP
- U8, U9: value MCP3008BIS -> MCP3008; symbol MCP3008BIS -> MCP3008
Connections:
- wire segments 194 -> 202
Other:
- note added: "A/D Module"
- moved on the sheet: C17, C18, C19, C3, C4, D2, J1, JP1, P1, R1, R13, R16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

Commit message: Schematic: split analog part
Parts:
- removed C14, C15, C16: 100n, Capacitors_SMD:C_0603, symbol C_Small
- removed C17, C18, C19: 47p, Capacitors_SMD:C_0603, symbol C_Small
- removed R16, R17, R18: 51k, Capacitors_SMD:C_0603, symbol R_Small
- removed R19, R20, R21, R22, R23, R24, R25, R26, R27: 1k, Capacitors_SMD:C_0603, symbol R_Small
- removed R28, R29, R30: 220, Capacitors_SMD:C_0603, symbol R_Small
- removed U10: Airspeed, SMD_Packages:SOIC-8-N, symbol MPXV5004DP
- removed U11: Static Pressure, SMD_Packages:SOIC-8-N, symbol MPXA6115A
- removed U12: MAP Pressure, SMD_Packages:SOIC-8-N, symbol MPXA6115A
- removed U8, U9: MCP3008, SMD_Packages:SO-16-L, symbol MCP3008
- C10: value 10nF -> 10n
- C12, C13: value 0.1uF -> 0.1u
Connections:
- net labels removed: ASI, BARO, CHT, MAP, MCP0_ADDR, MCP1_ADDR, OilPressure, OilTemp
- wire segments 202 -> 147
- no-connect marks 50 -> 43
Other:
- note removed: "A/D Module"
- note removed: "Pressure Module"
- moved on the sheet: D4, D5

Commit message: Schematic work
Parts:
- removed D4: Diode, Diodes_SMD:D_0603, symbol D_Small
- removed D5: 3.3V, Diodes_SMD:D_SOD-323, symbol D_Zener_Small
- removed J2: Screw_Terminal_1x12, Connectors_Terminal_Blocks:TerminalBlock_Pheonix_MPT-2.54mm_12pol, symbol Screw_Terminal_1x12
- removed R14: 10k, Resistors_SMD:R_0603, symbol R_Small
- removed R15: 100k, Resistors_SMD:R_0603, symbol R_Small
Connections:
- net labels removed: TACH, TACH_IN
- wire segments 147 -> 138
- no-connect marks 43 -> 32
Other:
- note removed: "Tachymeter Module"
Changed lines of the file:
@@
 	0    -1   -1   0
 $EndComp
-$Comp
-L Screw_Terminal_1x12 J2
-U 1 1 58CC8F45
-P 15700 3150
-F 0 "J2" H 15700 4400 50  0000 C TNN
-F 1 "Screw_Terminal_1x12" V 15550 3150 50  0000 C TNN
-F 2 "Connectors_Terminal_Blocks:TerminalBlock_Pheonix_MPT-2.54mm_12pol" H 15700 1925 50  0001 C CNN
-F 3 "" H 15675 4150 50  0001 C CNN
-	1    15700 3150
-	-1   0    0    1
-$EndComp
-$Comp
-L D_Small D4
-U 1 1 58CC93C1
-P 10050 10330
-F 0 "D4" H 10000 10410 50  0000 L CNN
-F 1 "Diode" H 9900 10250 50  0000 L CNN
-F 2 "Diodes_SMD:D_0603" V 10050 10330 50  0001 C CNN
-F 3 "" V 10050 10330 50  0001 C CNN
-	1    10050 10330
-	0    1    1    0
-$EndComp
-$Comp
-L D_Zener_Small D5
-U 1 1 58CC9DAC
-P 10550 10330
-F 0 "D5" H 10550 10420 50  0000 C CNN
-F 1 "3.3V" H 10550 10240 50  0000 C CNN
-F 2 "Diodes_SMD:D_SOD-323" V 10550 10330 50  0001 C CNN
-F 3 "" V 10550 10330 50  0001 C CNN
-	1    10550 10330
-	0    1    1    0
-$EndComp
-$Comp
-L R_Small R15
-U 1 1 58CC9EF8
-P 10300 10150
-F 0 "R15" H 10330 10170 50  0000 L CNN
-F 1 "100k" H 10330 10110 50  0000 L CNN
-F 2 "Resistors_SMD:R_0603" H 10300 10150 50  0001 C CNN
-F 3 "" H 10300 10150 50  0001 C CNN
-	1    10300 10150
-	0    1    1    0
-$EndComp
-$Comp
-L R_Small R14
-U 1 1 58CCA086
-P 9800 10150
-F 0 "R14" H 9830 10170 50  0000 L CNN
-F 1 "10k" H 9830 10110 50  0000 L CNN
-F 2 "Resistors_SMD:R_0603" H 9800 10150 50  0001 C CNN
-F 3 "" H 9800 10150 50  0001 C CNN
-	1    9800 10150
-	0    1    1    0
-$EndComp
-$Comp
-L GND #PWR028
-U 1 1 58CCA77F
-P 10300 10600
-F 0 "#PWR028" H 10300 10600 30  0001 C CNN
-F 1 "GND" H 10300 10530 30  0001 C CNN
-F 2 "" H 10300 10600 60  0001 C CNN
-F 3 "" H 10300 10600 60  0001 C CNN
-	1    10300 10600
-	1    0    0    -1
-$EndComp
-Text Label 9550 10150 2    60   ~ 0
-TACH_IN
-Text Label 10700 10150 0    60   ~ 0
-TACH
-Text Notes 9000 10900 0    157  Italic 31
-Tachymeter Module
-Text Label 15500 2050 2    60   ~ 0
-TACH_IN
-NoConn ~ 15500 2850
-NoConn ~ 15500 3050
-NoConn ~ 15500 3250
-NoConn ~ 15500 3450
-NoConn ~ 15500 3650
-NoConn ~ 15500 3850
-NoConn ~ 15500 4050
-NoConn ~ 15500 4250
 Text Label 7100 8300 0    60   ~ 0
 +3.3V
@@
 +5V
 $Comp
-L PWR_FLAG #FLG029
+L PWR_FLAG #FLG028
 U 1 1 58CE60AD
 P 4550 7150
-F 0 "#FLG029" H 4550 7225 50  0001 C CNN
+F 0 "#FLG028" H 4550 7225 50  0001 C CNN
 F 1 "PWR_FLAG" H 4550 7300 50  0000 C CNN
 F 2 "" H 4550 7150 50  0001 C CNN
@@
 $EndComp
 $Comp
-L PWR_FLAG #FLG030
+L PWR_FLAG #FLG029
 U 1 1 58CE6314
 P 5100 7150
-F 0 "#FLG030" H 5100 7225 50  0001 C CNN
+F 0 "#FLG029" H 5100 7225 50  0001 C CNN
 F 1 "PWR_FLAG" H 5100 7300 50  0000 C CNN
 F 2 "" H 5100 7150 50  0001 C CNN
@@
 $EndComp
 Wire Wire Line
-	10550 10500 10550 10430
-Wire Wire Line
-	10050 10430 10050 10500
-Wire Wire Line
 	6000 7100 6000 7150
 Wire Wire Line
@@
 	5700 6300 5800 6300
 Wire Wire Line
-	10050 10500 10550 10500
-Wire Wire Line
-	10300 10500 10300 10600
-Connection ~ 10300 10500
-Wire Wire Line
-	9900 10150 10200 10150
-Wire Wire Line
-	10050 10230 10050 10150
-Connection ~ 10050 10150
-Wire Wire Line
-	10400 10150 10700 10150
-Wire Wire Line
-	10550 10230 10550 10150
-Connection ~ 10550 10150
-Wire Wire Line
-	9700 10150 9550 10150
-Wire Notes Line
-	8850 10000 11450 10000
-Wire Notes Line
-	11450 10000 11450 11000
-Wire Notes Line
-	11450 11000 8850 11000
-Wire Notes Line
-	8850 11000 8850 10000
-Wire Wire Line
 	6900 8300 6900 8600
 Wire Wire Line
@@
 Wire Wire Line
 	7200 3200 9280 3200
-NoConn ~ 15500 2250
-NoConn ~ 15500 2450
-NoConn ~ 15500 2650
 Text Label 7200 2800 0    60   ~ 0
 MOSI

Commit message: Another RPM reading solution
Connections:
- net Analog Sensors/TACH: now also P3.22 (GPIO25); no longer P3.31 (GPIO6)
- no-connect marks 32 -> 31
Changed lines of the file:
@@
 $EndComp
 $Comp
-L GND #PWR01
+L GND #PWR11
 U 1 1 54E93493
 P 3900 5100
-F 0 "#PWR01" H 3900 5100 30  0001 C CNN
+F 0 "#PWR11" H 3900 5100 30  0001 C CNN
 F 1 "GND" H 3900 5030 30  0001 C CNN
 F 2 "" H 3900 5100 60  0000 C CNN
@@
 $EndComp
 $Comp
-L GND #PWR02
+L GND #PWR8
 U 1 1 54E93549
 P 2400 5100
-F 0 "#PWR02" H 2400 5100 30  0001 C CNN
+F 0 "#PWR8" H 2400 5100 30  0001 C CNN
 F 1 "GND" H 2400 5030 30  0001 C CNN
 F 2 "" H 2400 5100 60  0000 C CNN
@@
 $EndComp
 $Comp
-L GND #PWR03
+L GND #PWR13
 U 1 1 54E963F9
 P 4500 3600
-F 0 "#PWR03" H 4500 3600 30  0001 C CNN
+F 0 "#PWR13" H 4500 3600 30  0001 C CNN
 F 1 "GND" H 4500 3530 30  0001 C CNN
 F 2 "" H 4500 3600 60  0000 C CNN
@@
 $EndComp
 $Comp
-L GND #PWR04
+L GND #PWR6
 U 1 1 54E98C85
 P 1250 10750
-F 0 "#PWR04" H 1250 10750 30  0001 C CNN
+F 0 "#PWR6" H 1250 10750 30  0001 C CNN
 F 1 "GND" H 1250 10680 30  0001 C CNN
 F 2 "" H 1250 10750 60  0000 C CNN
@@
 $EndComp
 $Comp
-L GND #PWR05
+L GND #PWR9
 U 1 1 54E98DFB
 P 2750 10750
-F 0 "#PWR05" H 2750 10750 30  0001 C CNN
+F 0 "#PWR9" H 2750 10750 30  0001 C CNN
 F 1 "GND" H 2750 10680 30  0001 C CNN
 F 2 "" H 2750 10750 60  0000 C CNN
@@
 $EndComp
 $Comp
-L GND #PWR06
+L GND #PWR2
 U 1 1 54E99B35
 P 800 9600
-F 0 "#PWR06" H 800 9600 30  0001 C CNN
+F 0 "#PWR2" H 800 9600 30  0001 C CNN
 F 1 "GND" H 800 9530 30  0001 C CNN
 F 2 "" H 800 9600 60  0000 C CNN
@@
 $EndComp
 $Comp
-L GND #PWR07
+L GND #PWR15
 U 1 1 54E9A81E
 P 4750 10750
-F 0 "#PWR07" H 4750 10750 30  0001 C CNN
+F 0 "#PWR15" H 4750 10750 30  0001 C CNN
 F 1 "GND" H 4750 10680 30  0001 C CNN
 F 2 "" H 4750 10750 60  0000 C CNN
@@
 $EndComp
 $Comp
-L +24V #PWR08
+L +24V #PWR1
 U 1 1 54F050C6
 P 800 8700
-F 0 "#PWR08" H 800 8650 20  0001 C CNN
+F 0 "#PWR1" H 800 8650 20  0001 C CNN
 F 1 "+24V" H 800 8850 30  0000 C CNN
 F 2 "" H 800 8700 60  0000 C CNN
@@
 $EndComp
 $Comp
-L GND #PWR09
+L GND #PWR7
 U 1 1 54F37150
 P 1600 8550
-F 0 "#PWR09" H 1600 8550 30  0001 C CNN
+F 0 "#PWR7" H 1600 8550 30  0001 C CNN
 F 1 "GND" H 1600 8480 30  0001 C CNN
 F 2 "" H 1600 8550 60  0000 C CNN
@@
 $EndComp
 $Comp
-L GND #PWR010
+L GND #PWR3
 U 1 1 54F379A8
 P 850 7950
-F 0 "#PWR010" H 850 7950 30  0001 C CNN
+F 0 "#PWR3" H 850 7950 30  0001 C CNN
 F 1 "GND" H 850 7880 30  0001 C CNN
 F 2 "" H 850 7950 60  0000 C CNN
@@
 $EndComp
 $Comp
-L GND #PWR011
+L GND #PWR10
 U 1 1 54F3D72C
 P 3400 8000
-F 0 "#PWR011" H 3400 8000 30  0001 C CNN
+F 0 "#PWR10" H 3400 8000 30  0001 C CNN
 F 1 "GND" H 3400 7930 30  0001 C CNN
 F 2 "" H 3400 8000 60  0000 C CNN
@@
 $EndComp
 $Comp
-L GND #PWR012
+L GND #PWR12
 U 1 1 54F4127D
 P 4050 8500
-F 0 "#PWR012" H 4050 8500 30  0001 C CNN
+F 0 "#PWR12" H 4050 8500 30  0001 C CNN
 F 1 "GND" H 4050 8430 30  0001 C CNN
 F 2 "" H 4050 8500 60  0000 C CNN
@@
 $EndComp
 $Comp
-L +24V #PWR013
+L +24V #PWR4
 U 1 1 54F662FB
 P 1050 6150
-F 0 "#PWR013" H 1050 6100 20  0001 C CNN
+F 0 "#PWR4" H 1050 6100 20  0001 C CNN
 F 1 "+24V" H 1050 6300 30  0000 C CNN
 F 2 "" H 1050 6150 60  0000 C CNN
@@
 $EndComp
 $Comp
-L GND #PWR014
+L GND #PWR5
 U 1 1 54F66353
 P 1050 6550
-F 0 "#PWR014" H 1050 6550 30  0001 C CNN
+F 0 "#PWR5" H 1050 6550 30  0001 C CNN
 F 1 "GND" H 1050 6480 30  0001 C CNN
 F 2 "" H 1050 6550 60  0000 C CNN
@@
 NoConn ~ 6450 6500
 $Comp
-L GND #PWR015
+L GND #PWR19
 U 1 1 58BCBCD4
 P 6000 7150
-F 0 "#PWR015" H 6000 6900 50  0001 C CNN
+F 0 "#PWR19" H 6000 6900 50  0001 C CNN
 F 1 "GND" H 6000 7000 50  0000 C CNN
 F 2 "" H 6000 7150 50  0001 C CNN
@@
 $EndComp
 $Comp
-L GND #PWR016
+L GND #PWR18
 U 1 1 58BCBCD5
 P 5950 6600
-F 0 "#PWR016" H 5950 6350 50  0001 C CNN
+F 0 "#PWR18" H 5950 6350 50  0001 C CNN
 F 1 "GND" H 5950 6450 50  0000 C CNN
 F 2 "" H 5950 6600 50  0001 C CNN
@@
 $EndComp
 $Comp
-L GND #PWR017
+L GND #PWR24
 U 1 1 58BCBCD6
 P 8400 6500
-F 0 "#PWR017" H 8400 6250 50  0001 C CNN
+F 0 "#PWR24" H 8400 6250 50  0001 C CNN
 F 1 "GND" H 8400 6350 50  0000 C CNN
 F 2 "" H 8400 6500 50  0001 C CNN
@@
 $EndComp
 $Comp
-L GND #PWR018
+L GND #PWR25
 U 1 1 58BCBCD7
 P 8400 7200
-F 0 "#PWR018" H 8400 6950 50  0001 C CNN
+F 0 "#PWR25" H 8400 6950 50  0001 C CNN
 F 1 "GND" H 8400 7050 50  0000 C CNN
 F 2 "" H 8400 7200 50  0001 C CNN
@@
 $EndComp
 $Comp
-L GND #PWR019
+L GND #PWR23
 U 1 1 58BCBCDC
 P 8100 7550
-F 0 "#PWR019" H 8100 7300 50  0001 C CNN
+F 0 "#PWR23" H 8100 7300 50  0001 C CNN
 F 1 "GND" H 8100 7400 50  0000 C CNN
 F 2 "" H 8100 7550 50  0001 C CNN
@@
 NoConn ~ 7850 7100
 $Comp
-L PWR_FLAG #FLG020
+L PWR_FLAG #FLG1
 U 1 1 58BD447B
 P 4550 6700
-F 0 "#FLG020" H 4550 6775 50  0001 C CNN
+F 0 "#FLG1" H 4550 6775 50  0001 C CNN
 F 1 "PWR_FLAG" H 4550 6850 50  0000 C CNN
 F 2 "" H 4550 6700 50  0001 C CNN
@@
 $EndComp
 $Comp
-L PWR_FLAG #FLG021
+L PWR_FLAG #FLG3
 U 1 1 58BD44DD
 P 5100 6700
-F 0 "#FLG021" H 5100 6775 50  0001 C CNN
+F 0 "#FLG3" H 5100 6775 50  0001 C CNN
 F 1 "PWR_FLAG" H 5100 6850 50  0000 C CNN
 F 2 "" H 5100 6700 50  0001 C CNN
@@
 $EndComp
 $Comp
-L GND #PWR022
+L GND #PWR16
 U 1 1 58BD4648
 P 5100 6700
-F 0 "#PWR022" H 5100 6700 30  0001 C CNN
+F 0 "#PWR16" H 5100 6700 30  0001 C CNN
 F 1 "GND" H 5100 6630 30  0001 C CNN
 F 2 "" H 5100 6700 60  0000 C CNN
@@
 $EndComp
 $Comp
-L +24V #PWR023
+L +24V #PWR14
 U 1 1 58BD46C2
 P 4550 6700
-F 0 "#PWR023" H 4550 6650 20  0001 C CNN
+F 0 "#PWR14" H 4550 6650 20  0001 C CNN
 F 1 "+24V" H 4550 6850 30  0000 C CNN
 F 2 "" H 4550 6700 60  0000 C CNN
@@
 NoConn ~ 7200 5200
 NoConn ~ 7200 5100
-NoConn ~ 7200 5000
 NoConn ~ 7200 4900
 NoConn ~ 7200 4800
@@
 RXD
 $Comp
-L GND #PWR024
+L GND #PWR17
 U 1 1 58BDF5E8
 P 5750 7750
-F 0 "#PWR024" H 5750 7500 50  0001 C CNN
+F 0 "#PWR17" H 5750 7500 50  0001 C CNN
 F 1 "GND" H 5750 7600 50  0000 C CNN
 F 2 "" H 5750 7750 50  0001 C CNN
@@
 SCLK
 $Comp
-L GND #PWR025
+L GND #PWR21
 U 1 1 58BEF3EB
 P 7000 10600
-F 0 "#PWR025" H 7000 10600 30  0001 C CNN
+F 0 "#PWR21" H 7000 10600 30  0001 C CNN
 F 1 "GND" H 7000 10530 30  0001 C CNN
 F 2 "" H 7000 10600 60  0000 C CNN
@@
 $EndComp
 $Comp
-L GND #PWR026
+L GND #PWR20
 U 1 1 58C81FE8
 P 6200 8800
-F 0 "#PWR026" H 6200 8800 30  0001 C CNN
+F 0 "#PWR20" H 6200 8800 30  0001 C CNN
 F 1 "GND" H 6200 8730 30  0001 C CNN
 F 2 "" H 6200 8800 60  0000 C CNN
@@
 $EndComp
 $Comp
-L GND #PWR027
+L GND #PWR22
 U 1 1 58C82484
 P 7750 8800
-F 0 "#PWR027" H 7750 8800 30  0001 C CNN
+F 0 "#PWR22" H 7750 8800 30  0001 C CNN
 F 1 "GND" H 7750 8730 30  0001 C CNN
 F 2 "" H 7750 8800 60  0000 C CNN
@@
 +5V
 $Comp
-L PWR_FLAG #FLG028
+L PWR_FLAG #FLG2
 U 1 1 58CE60AD
 P 4550 7150
-F 0 "#FLG028" H 4550 7225 50  0001 C CNN
+F 0 "#FLG2" H 4550 7225 50  0001 C CNN
 F 1 "PWR_FLAG" H 4550 7300 50  0000 C CNN
 F 2 "" H 4550 7150 50  0001 C CNN
@@
 $EndComp
 $Comp
-L PWR_FLAG #FLG029
+L PWR_FLAG #FLG4
 U 1 1 58CE6314
 P 5100 7150
-F 0 "#FLG029" H 5100 7225 50  0001 C CNN
+F 0 "#FLG4" H 5100 7225 50  0001 C CNN
 F 1 "PWR_FLAG" H 5100 7300 50  0000 C CNN
 F 2 "" H 5100 7150 50  0001 C CNN
@@
 	9280 3300 7770 3300
 Wire Wire Line
-	7770 3300 7770 3800
-Wire Wire Line
-	7770 3800 7200 3800
+	7770 3300 7770 5000
+Wire Wire Line
+	7770 5000 7200 5000
 $EndSCHEMATC

Commit message: Work on schematic
Parts:
- added J?: CONN_01X03, symbol CONN_01X03
- added Q?: BSS138, TO_SOT_Packages_SMD:SOT-23, symbol BSS138
- added R? (x2): 10k, symbol R
Connections:
- net +3.3V: now also Q?.1 (G), R?.1
- net +5V: now also J?.3 (P3), R?.1
- net Analog Sensors/TACH: no longer P3.22 (GPIO25)
- net GND: now also J?.1 (P1)
- net Fuel_Flow: now reaches P3.32 (GPIO12)
- net Fuel_Flow: now also Q?.2 (S), R?.2
- new net: J?.2 (P2), Q?.3 (D), R?.2
- no-connect marks 31 -> 30

Commit message: Clear PCB network + clean schematic
Parts:
- J2: renamed from J?; footprint (none) -> Pin_Headers:Pin_Header_Straight_1x03_Pitch2.00mm
- R21, R22: renamed from R?; footprint (none) -> Resistors_SMD:R_0603
- gave numbers to parts that had none: 1
Connections:
- net Analog Sensors/TACH: now also P3.31 (GPIO6)
- net GND: now also J2.2 (P2); no longer J2.1 (P1)
- net MISO: no longer U7.9 (AD0/MISO)
- net MOSI: no longer U7.24 (SDA/MOSI)
- net SCLK: no longer U7.23 (SCL/SCLK)
- net I2C_SDA: now reaches P3.3 (GPIO2/I2C1_SDA)
- net I2C_SDA: now also U7.24 (SDA/MOSI)
- net I2C_SCLK: now reaches P3.5 (GPIO3/I2C1_SCL)
- net I2C_SCLK: now also U7.23 (SCL/SCLK)
- net at Q2.3 (D), R21.2: now also J2.1 (P1); no longer J2.2 (P2)
- net MPU0_ADDR: no longer names the net of P3.29 (GPIO5)
- net MPU0_ADDR: no longer U7.22 (~CS)
- net MPU0_INT: no longer names the net of P3.7 (GPIO4/GPCLK0)
- net MPU0_INT: no longer U7.12 (INT)
- no-connect marks 30 -> 34
Other:
- moved on the sheet: Q2, R21, R22

Commit message: Work on circuit & PCB
Parts:
- removed C1: 50uf/50v, w_smd_cap:c_elec_6.3x7.7, symbol CP
- removed C2, C5: 0.1uf, Capacitors_SMD:C_0603, symbol C
- removed C6: 10uf/6.3V, Capacitors_SMD:CP_Elec_4x5.3, symbol CP
- removed C8: 1uf, Capacitors_SMD:C_0603, symbol C
- removed D1: DIODESCH, w_smd_diode:do214aa, symbol D_Schottky
- removed D3: LED, Diodes_SMD:D_0603, symbol LED-RESCUE-pihat_template
- removed L1: 22uH, w_smd_inductors:inductor_smd_8x5mm, symbol INDUCTOR-RESCUE-pihat_template
- removed R10: 360, Resistors_SMD:R_0603, symbol R
- removed R2: 24k, Resistors_SMD:R_0603, symbol R
- removed R4: 270, Resistors_SMD:R_0603, symbol R
- removed R6: 30k, Resistors_SMD:R_0603, symbol R
- removed R7: 10k, Resistors_SMD:R_0603, symbol R
- removed R8: 390, Resistors_SMD:R_0603, symbol R
- removed R9: 240, Resistors_SMD:R_0603, symbol R
- removed U1: LM3489, w_smd_dil:msoic-8, symbol LM3489
- removed U3: FDC5614P, w_smd_trans:sot23-6, symbol FDC5614P
- removed U4: LM1117IMPX-ADJ, w_smd_trans:sot223, symbol LM1117IMPX-ADJ
- added C1, C5: 100n, Capacitors_SMD:C_0603, symbol C_Small
- added C14, C16: 1u, Capacitors_SMD:C_0603, symbol C_Small
- added C17, C20: 0.01u, Capacitors_SMD:C_0603, symbol C_Small
- added C19: 0.1u, Capacitors_SMD:C_0603, symbol C
- added C21: 470p, Capacitors_SMD:C_0603, symbol C_Small
- added C23: 47p, Capacitors_SMD:C_0603, symbol C_Small
- added C24: 22n, Capacitors_SMD:C_0603, symbol C_Small
- added D4: Diode, Diodes_SMD:D_0603, symbol D_Small
- added D5: 5.6V, Diodes_SMD:D_SOD-323, symbol D_Zener_Small
- added J3: CONN_01X04, Pin_Headers:Pin_Header_Straight_1x04_Pitch2.54mm, symbol CONN_01X04
- added J4, J5: CONN_01X03, Pin_Headers:Pin_Header_Straight_1x03_Pitch2.54mm, symbol CONN_01X03
- added P4: CONN_01X02, Pin_Headers:Pin_Header_Straight_1x02_Pitch2.54mm, symbol CONN_01X02
- added Q3, Q4, Q5: BSS138, TO_SOT_Packages_SMD:SOT-23, symbol BSS138
- added R14, R27: 10k, Resistors_SMD:R_0603, symbol R_Small
- added R15, R20, R23: 220, Resistors_SMD:R_0603, symbol R_Small
- added R16, R26: 100k, Resistors_SMD:R_0603, symbol R_Small
- added R17: 47k, Resistors_SMD:R_0603, symbol R_Small
- added R19: 51k, Resistors_SMD:R_0603, symbol R_Small
- added R24, R25, R28, R29, R30, R31: 10k, Resistors_SMD:R_0603, symbol R
- added U1: MIC5219-3.3BM5, TO_SOT_Packages_SMD:SOT-23-5, symbol MIC5219-3.3BM5
- added U11: MAP Pressure, SMD_Packages:SOIC-8-N, symbol MPXA6115A
- added U12: LM358, Housings_SOIC:SOIC-8_3.9x4.9mm_Pitch1.27mm, symbol LM358
- added U3: BME280, aeroPi:BME280, symbol BME280
- added U8: Airspeed, SMD_Packages:SOIC-8-N, symbol MPXV5004DP
- added U9: ADS7828, Housings_SSOP:TSSOP-16_4.4x5mm_Pitch0.65mm, symbol ADS7828
- C3: value 1nf -> 10u; Mouser Part No. 810-C1005C0G2A102J5C -> (none)
- C7: value 0.1uf -> 10u; Mouser Part No. 810-C1005X5R1H104K -> (none)
- J2: footprint Pin_Headers:Pin_Header_Straight_1x03_Pitch2.00mm -> Pin_Headers:Pin_Header_Straight_1x03_Pitch2.54mm
- P1: footprint w_pin_strip:pin_strip_2 -> Pin_Headers:Pin_Header_Straight_1x02_Pitch2.54mm
- P2: footprint w_conn_mkds:mkds_1,5-2 -> Pin_Headers:Pin_Header_Straight_1x02_Pitch2.54mm
- P3: footprint w_conn_strip:vasch_strip_20x2 -> w_pin_strip:pin_socket_20x2
Connections:
- net +3.3V: now also U7.22 (~CS), C1.1, C5.1, Q3.1 (G), Q4.1 (G), Q5.1 (G), R25.1, R29.1, R31.1, U1.5 (VOUT), U3.2 (CSB), U3.6 (VDDIO), U3.8 (VDD)
- net +5V: now also C3.1, P2.2 (P2), C14.1, C16.1, C17.1, C19.1, C20.1, J4.3 (P3), J5.3 (P3), R15.2, R20.2, R23.1, R24.1, R26.2, R28.1, R30.1, U1.1 (VIN), U1.3 (EN), U11.2 (Vcc), U12.8 (V+), U12.8 (V+), U8.2 (Vcc), U9.10 (REF), U9.16 (VDD)
- net Fuel_Flow: now also P3.22 (GPIO25), Q5.2 (S), R31.2; no longer P3.32 (GPIO12), Q2.2 (S), R22.2
- net GND: now also C3.2, P2.1 (P1), U7.9 (AD0/MISO), C1.2, C14.2, C16.2, C17.2, C19.2, C20.2, C21.2, C23.2, C24.2, C5.2, D4.2 (A), D5.2 (A), J4.1 (P1), J5.1 (P1), P4.1 (P1), R19.2, R27.1, U1.2 (GND), U11.3 (GND), U12.4 (V-), U12.4 (V-), U3.1 (GND), U3.5 (SDO), U3.7 (GND), U8.3 (GND), U9.11 (COM), U9.12 (A0), U9.13 (A1), U9.9 (GND); no longer P2.2 (P2)
- net I2C_SCLK: now also Q3.2 (S), R25.2, U3.4 (SCK)
- net I2C_SDA: now also Q2.2 (S), R22.2, U3.3 (SDI)
- net 1PPS: now reaches P3.29 (GPIO5)
- net 1PPS: now also U6.13 (1PPS)
- net Tach: now reaches P3.7 (GPIO4/GPCLK0)
- net Tach: now also Q4.2 (S), R29.2
- net at Q2.3 (D), R21.2: now also U9.15 (SDA); no longer J2.1 (P1)
- removed net +24V: C3.1, P2.1 (P1)
- net Analog Sensors/MCP0_ADDR: no longer names the net of P3.24 (GPIO8/SPI_CE0)
- net Analog Sensors/MCP1_ADDR: no longer names the net of P3.26 (GPIO7/SPI_CE1)
- net Analog Sensors/TACH: no longer names the net of P3.31 (GPIO6)
- net MISO: no longer names the net of P3.21 (GPIO9/SPI_MISO)
- net MOSI: no longer names the net of P3.19 (GPIO10/SPI_M0SI)
- net SCLK: no longer names the net of P3.23 (GPIO11/SPI_SCLK)
- new net: J2.1 (P1), Q5.3 (D), R30.2
- new net: Q3.3 (D), R24.2, U9.14 (SCL)
- new net: Q4.3 (D), R28.2, U12.7
- new net: D4.1 (K), R14.1, R16.2
- new net: D5.1 (K), R16.1, R17.2
- new net: C24.1, R17.1, U12.3 (+)
- new net: U12.1, U12.2 (-), U12.5 (+)
- new net: R26.1, R27.2, U12.6 (-)
- new net +5VRpi: P4.2 (P2)
- new net ASI: C21.1, U8.4 (Vout), U9.6 (CH5)
- new net CHT: J3.2 (P2), R15.1, U9.3 (CH2)
- new net CurrentMeter: J4.2 (P2), U9.4 (CH3)
- new net MAP: C23.1, R19.1, U11.4 (Vout), U9.7 (CH6)
- new net OilPressure: J3.4 (P4), R23.2, U9.1 (CH0)
- new net OilTemp: J3.3 (P3), R20.1, U9.2 (CH1)
- new net Tachometer: J3.1 (P1), R14.2
- new net VoltageMeter: J5.2 (P2), U9.5 (CH4)
- no-connect marks 34 -> 36
Other:
- note added: "3v3 @ 0.5A DC/DC supply for 3v3 sensors"
- note added: "A/D Module"
- note added: "Capacitor C14,C16,C17,C18 and C19 must be as close as \npossible to the VCC pin of each sensor on the PCB"
- note added: "Pressure Module"
- note added: "Tachometer Module"
- note removed: "3.3v @ 1.5A LDO supply"
- note removed: "5v @ 2.1A DC/DC supply"
- moved on the sheet: BT1, C10, C11, C12, C13, C9, D2, J1, J2, L2, P2, Q2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

Commit message: Work on circuit and add documentation + 3D model
Parts:
- removed C4: 0.1uf, Capacitors_SMD:C_0603, symbol C
- removed J2, J4, J5: CONN_01X03, Pin_Headers:Pin_Header_Straight_1x03_Pitch2.54mm, symbol CONN_01X03
- removed J3: CONN_01X04, Pin_Headers:Pin_Header_Straight_1x04_Pitch2.54mm, symbol CONN_01X04
- removed JP1: JUMPER, Resistors_SMD:R_0603, symbol JUMPER-RESCUE-pihat_template
- removed P1: CONN_01X02, Pin_Headers:Pin_Header_Straight_1x02_Pitch2.54mm, symbol CONN_01X02
- removed R1: 1k, Resistors_SMD:R_0603, symbol R
- removed R3, R5: 3.9k, Resistors_SMD:R_0603, symbol R
- removed U2: CAT24C32HU4I-GT3, w_smd_dil:tssop-8, symbol CAT24C32HU4I-GT3
- added D1: 1N4148, Diodes_SMD:D_SOD-323, symbol D_Small
- added J2: DB15_FEMALE, Connectors:DB15FC, symbol DB15_FEMALE
- added J4: CONN_01X04, Pin_Headers:Pin_Header_Straight_1x04_Pitch2.54mm, symbol CONN_01X04
- added R1: 10K, Resistors_SMD:R_0603, symbol R_Small
- BT1: footprint Connectors:CR1220 -> Battery_Holders:Keystone_3000_1x12mm-CoinCell
- D4: value Diode -> 1N4007; footprint Diodes_SMD:D_0603 -> Diodes_SMD:D_SOD-323
- Q2, Q3, Q4, Q5: symbol BSS138 -> BSS138-RESCUE-aeroPi
- U11: footprint SMD_Packages:SOIC-8-N -> aeroPi:MPXA6115A
- U8: footprint SMD_Packages:SOIC-8-N -> aeroPi:MPXV5004DP
Connections:
- net Back Power Protection/5V_MCU is gone; now on net +5VRpi: P3.2 (VPP_(5v)), P3.4 (VPP_(5v))
- net +3.3V: now also J4.3 (P3), R1.2
- net +5V: now also J2.12 (P12), J2.13 (P13)
- net 1PPS: now also P3.7 (GPIO4/GPCLK0); no longer P3.29 (GPIO5)
- net CHT: now also J2.5
- net CurrentMeter: now also J2.4
- net Fuel_Flow: now also P3.11 (GPIO17); no longer P3.22 (GPIO25)
- net GND: now also J2.10 (P10), J2.11 (P111), J2.14 (P14), J4.4 (P4)
- net I2C_SCLK: now also J4.1 (P1)
- net I2C_SDA: now also J4.2 (P2)
- net OilPressure: now also J2.7
- net OilTemp: now also J2.6
- net RXD: now also D1.1 (K), J2.15 (P15); no longer U6.9 (TX)
- net TXD: now also U6.9 (TX), J2.8; no longer U6.10 (RX)
- net Tach: now also P3.12 (GPIO18); no longer P3.7 (GPIO4/GPCLK0)
- net Tachometer: now also J2.1
- net VoltageMeter: now also J2.3
- net Fuel_Flow_In: now reaches Q5.3 (D), R30.2
- net Fuel_Flow_In: now also J2.2
- net AirTemp: now reaches U9.8 (CH7)
- net AirTemp: now also J2.9 (P9)
- new net: D1.2 (A), R1.1, U6.10 (RX)
- no-connect marks 36 -> 37
Other:
- note added: "I²C : 0x48"
- note added: "I²C : 0x68 + 0x0C"
- note added: "I²C : 0x76"
- moved on the sheet: BT1, C14, C17, C21, Q5, R30, R31, U8
