File: resources/circuit/aeroPi.sch (KiCad schematic (older format))
At the start: 60 parts, among them J1 CONN_COAXIAL, J2 DB15_FEMALE, J4 CONN_01X04, P2 CONN_01X02, P3 Raspberry_Pi_+_Conn, P4 CONN_01X02, Q2 BSS138, Q3 BSS138, Q4 BSS138, Q5 BSS138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

Commit message: schema wip
Parts:
- R27: value 10k -> 47k
Changed lines of the file:
@@
 EESchema Schematic File Version 2
 LIBS:aeroPi-rescue
-LIBS:power
-LIBS:device
-LIBS:transistors
-LIBS:conn
-LIBS:linear
-LIBS:regul
-LIBS:74xx
-LIBS:cmos4000
-LIBS:adc-dac
-LIBS:memory
-LIBS:xilinx
-LIBS:microcontrollers
-LIBS:dsp
-LIBS:microchip
-LIBS:analog_switches
-LIBS:motorola
-LIBS:texas
-LIBS:intel
-LIBS:audio
-LIBS:interface
-LIBS:digital-audio
-LIBS:philips
-LIBS:display
-LIBS:cypress
-LIBS:siliconi
-LIBS:opto
-LIBS:atmel
-LIBS:contrib
-LIBS:valves
 LIBS:aeroPi
 LIBS:bme280
@@
 P 9240 10690
 F 0 "R27" H 9270 10710 50  0000 L CNN
-F 1 "10k" H 9270 10650 50  0000 L CNN
+F 1 "47k" H 9270 10650 50  0000 L CNN
 F 2 "Resistors_SMD:R_0603" H 9240 10690 50  0001 C CNN
 F 3 "" H 9240 10690 50  0001 C CNN

Commit message: Add electronic data
Parts:
- BT1: symbol Battery_Cell -> aeroPi:Battery_Cell
- C1, C14, C16, C17, C20, C21, C23, C24, C5: symbol C_Small -> aeroPi:C_Small
- C10, C11, C12, C13, C19, C3, C7, C9: symbol C -> aeroPi:C
- D1, D4: symbol D_Small -> aeroPi:D_Small
- D2: symbol LED_Small -> aeroPi:LED_Small
- D5: symbol D_Zener_Small -> aeroPi:D_Zener_Small
- J1: symbol CONN_COAXIAL -> aeroPi:CONN_COAXIAL
- J2: symbol DB15_FEMALE -> aeroPi-rescue:DB15_FEMALE
- J4: symbol CONN_01X04 -> aeroPi-rescue:CONN_01X04
- L2: symbol Ferrite_Bead_Small -> aeroPi:Ferrite_Bead_Small
- P2, P4: symbol CONN_01X02 -> aeroPi:CONN_01X02
- P3: symbol Raspberry_Pi_+_Conn -> aeroPi:Raspberry_Pi_+_Conn
- Q2, Q3, Q4, Q5: symbol BSS138-RESCUE-aeroPi -> aeroPi-rescue:BSS138-RESCUE-aeroPi
- R1, R13, R14, R15, R16, R17, R19, R20, R23, R26, R27: symbol R_Small -> aeroPi:R_Small
- R21, R22, R24, R25, R28, R29, R30, R31: symbol R -> aeroPi:R
- U1: symbol MIC5219-3.3BM5 -> aeroPi-rescue:MIC5219-3.3BM5
- U11: symbol MPXA6115A -> aeroPi:MPXA6115A
- U12: symbol LM358 -> aeroPi-rescue:LM358
- U3: symbol BME280 -> bme280:BME280
- U6: symbol FGPMMOPA6H -> aeroPi:FGPMMOPA6H
- U7: symbol MPU-9250 -> aeroPi:MPU-9250
- U8: symbol MPXV5004DP -> aeroPi:MPXV5004DP
- U9: symbol ADS7828 -> aeroPi-rescue:ADS7828
Connections:
- wire segments 190 -> 255
